File: RX_nrf24/_autosave-RX_nrf24.kicad_pcb (KiCad board)
At the start: 2 copper layers, 58.5 x 26.2 mm, 44 parts, among them J1 USB_B_Micro, J2 Conn_01x03_Male, J3 Conn_Coaxial, J4 Conn_01x10_Male, J5 Conn_01x04_Female, J6 Conn_01x06_Male, J7 Conn_01x10_Male, J8 Conn_01x10_Male, SW1 SW_Push, U1 USBLC6-2SC6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

Commit message: update pcb
Parts:
- C10, C11, C8: moved to B.Cu
- moved J2 12.3 mm to (157.1, 114.7)
- moved J5 12.3 mm to (167.6, 114.7)
- moved D1 12.3 mm to (172.4, 113.9)
- moved R3 12.3 mm to (172.3, 112.4)
- moved C4 8.42 mm to (151.5, 100.8)
- moved U2 8.42 mm to (155.6, 101.1)
- moved C5 8.42 mm to (153.2, 101.0)
- moved C9 8.42 mm to (158.5, 101.0)
- moved J1 7.65 mm to (154.4, 108.1)
- moved C8 5.32 mm to (170.2, 95.8)
- moved C11 5.22 mm to (170.2, 97.3)
- moved C10 4.92 mm to (163.8, 106.1)
- moved U1 4.87 mm to (164.1, 110.2)
- moved C7 4.52 mm to (175.1, 108.2)
- moved U3 4.52 mm to (170.4, 103.4)
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Routing:
- net P10: track 27.4 -> 9.01 mm
- net P9: track 24.6 -> 6.47 mm
- net P8: track 21.9 -> 6.04 mm
- net P7: track 19.5 -> 4.80 mm
- net P6: track 16.0 -> 5.26 mm
- net USB_D+: track 16.9 -> 9.10 mm
- net USB_D-: track 16.7 -> 9.09 mm
- net P5: track 12.2 -> 4.79 mm
- net RF_out: track 5.85 -> 12.0 mm
- net P4: track 9.60 -> 3.46 mm
- net +5V: track 9.24 -> 3.56 mm
- net P2: track 6.73 -> 1.27 mm
- net UART3_TX: track 3.75 -> 8.96 mm
- net UART3_RX: track 1.68 -> 6.09 mm
- net P1: track 7.49 -> 3.27 mm
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Other:
- board size 58.5 x 26.2 mm -> 58.6 x 30 mm
