File: RX_nrf24/RX_nrf24.sch (KiCad schematic (older format))
At the start: 55 parts, among them J1 USB_B_Micro, J2 Conn_01x03_Male, J3 Conn_Coaxial, J4 Conn_01x10_Male, J5 Conn_01x04_Female, J6 Conn_01x06_Male, SW1 SW_Push, U1 USBLC6-2SC6, U2 AMS1117-3.3, U3 STM32F103C8Tx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

Commit message: a
Parts:
- removed C13: CP, Capacitor_Tantalum_SMD:CP_EIA-3528-12_Kemet-T_Pad1.50x2.35mm_HandSolder, symbol Device:CP
- removed C15, C17, C18, C19, C21, C23, C24: C, Capacitor_SMD:C_0603_1608Metric_Pad1.05x0.95mm_HandSolder, symbol Device:C
- removed L1, L2: L, Capacitor_SMD:C_0603_1608Metric_Pad1.05x0.95mm_HandSolder, symbol Device:L
- removed R1: 1M, Resistor_SMD:R_0603_1608Metric_Pad1.05x0.95mm_HandSolder, symbol Device:R
- removed R4, R5: R, Resistor_SMD:R_0603_1608Metric_Pad1.05x0.95mm_HandSolder, symbol Device:R
- removed U2: AMS1117-3.3, Package_TO_SOT_SMD:SOT-223-3_TabPin2, symbol Regulator_Linear:AMS1117-3.3
- removed U4: RFX2401C, RF:QFN50P300X300X60-17N, symbol stm32_nrf24-rescue:RFX2401C-RFX2401C
- added J7, J8: Conn_01x10_Male, Connector_PinHeader_2.54mm:PinHeader_1x10_P2.54mm_Vertical, symbol Connector:Conn_01x10_Male
- added U2: MCP1700-3302E_SOT23, Package_TO_SOT_SMD:SOT-23, symbol Regulator_Linear:MCP1700-3302E_SOT23
- 1pF1, 1pF3: footprint Capacitor_SMD:C_0603_1608Metric -> Capacitor_SMD:C_0402_1005Metric
- C4, C9: footprint Capacitor_Tantalum_SMD:CP_EIA-3528-12_Kemet-T_Pad1.50x2.35mm_HandSolder -> Capacitor_SMD:C_1206_3216Metric
- J1: footprint Connector_USB:USB_Micro-B_GCT_USB3076-30-A -> Connector_USB:USB_Micro-B_Molex_47346-0001
- J3: footprint Connector_Coaxial:SMA_Amphenol_132289_EdgeMount -> Connector_Coaxial:SMA_Amphenol_132203-12_Horizontal
- SW1: footprint Button_Switch_THT:SW_PUSH_6mm_H5mm -> Button_Switch_SMD:SW_Push_1P1T_NO_6x6mm_H9.5mm
Connections:
- net labels added: UART3_CTS, UART3_RTS, UART3_RX, UART3_TX
- wire segments 210 -> 222
Other:
- moved on the sheet: J3, J6

Commit message: update pcb
Connections:
- net +5V: now also U1.5 (VBUS)
- net GND: now also U1.2 (GND)
Changed lines of the file:
@@
+	1    0    0    -1
+$EndComp
+Wire Wire Line
+	2550 6350 2550 6150
+$Comp
+L power:+5V #PWR?
+U 1 1 5F389BC7
+P 2550 6150
+F 0 "#PWR?" H 2550 6000 50  0001 C CNN
+F 1 "+5V" H 2565 6323 50  0000 C CNN
+F 2 "" H 2550 6150 50  0001 C CNN
+F 3 "" H 2550 6150 50  0001 C CNN
+	1    2550 6150
+	1    0    0    -1
+$EndComp
+$Comp
+L power:GND #PWR?
+U 1 1 5F39918F
+P 2550 7150
+F 0 "#PWR?" H 2550 6900 50  0001 C CNN
+F 1 "GND" H 2555 6977 50  0000 C CNN
+F 2 "" H 2550 7150 50  0001 C CNN
+F 3 "" H 2550 7150 50  0001 C CNN
+	1    2550 7150
 	1    0    0    -1
 $EndComp
