File: RX_nrf24/RX_nrf24.sch (KiCad schematic (older format))
At the start: 45 parts, among them J1 USB_B_Micro, J2 Conn_01x03_Male, J3 Conn_Coaxial, J4 Conn_01x10_Male, J5 Conn_01x04_Female, J6 Conn_01x06_Male, J7 Conn_01x10_Male, J8 Conn_01x10_Male, SW1 SW_Push, U1 USBLC6-2SC6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

Commit message: add alot
Parts:
- C1, C2: footprint Capacitor_SMD:C_0603_1608Metric_Pad1.05x0.95mm_HandSolder -> Capacitor_SMD:C_0402_1005Metric
- R1: renamed from R?; footprint (none) -> Resistor_SMD:R_0603_1608Metric
Changed lines of the file:
@@
 F 0 "C2" H 1465 2996 50  0000 L CNN
 F 1 "18pF" H 1465 2905 50  0000 L CNN
-F 2 "Capacitor_SMD:C_0603_1608Metric_Pad1.05x0.95mm_HandSolder" H 1388 2800 50  0001 C CNN
+F 2 "Capacitor_SMD:C_0402_1005Metric" H 1388 2800 50  0001 C CNN
 F 3 "~" H 1350 2950 50  0001 C CNN
 	1    1350 2950
@@
 F 0 "C1" H 1065 2996 50  0000 L CNN
 F 1 "18pF" H 1065 2905 50  0000 L CNN
-F 2 "Capacitor_SMD:C_0603_1608Metric_Pad1.05x0.95mm_HandSolder" H 988 2800 50  0001 C CNN
+F 2 "Capacitor_SMD:C_0402_1005Metric" H 988 2800 50  0001 C CNN
 F 3 "~" H 950 2950 50  0001 C CNN
 	1    950  2950
@@
 $EndComp
 $Comp
-L Device:R R?
+L Device:R R1
 U 1 1 5F97C2D0
 P 2100 7150
-F 0 "R?" H 2170 7196 50  0000 L CNN
+F 0 "R1" H 2170 7196 50  0000 L CNN
 F 1 "R" H 2170 7105 50  0000 L CNN
-F 2 "" V 2030 7150 50  0001 C CNN
+F 2 "Resistor_SMD:R_0603_1608Metric" V 2030 7150 50  0001 C CNN
 F 3 "~" H 2100 7150 50  0001 C CNN
 	1    2100 7150
@@
 	1650 7300 1650 7050
 $Comp
-L power:+3.3V #PWR?
+L power:+3.3V #PWR0124
 U 1 1 5F99EA10
 P 1650 7050
-F 0 "#PWR?" H 1650 6900 50  0001 C CNN
+F 0 "#PWR0124" H 1650 6900 50  0001 C CNN
 F 1 "+3.3V" H 1665 7223 50  0000 C CNN
 F 2 "" H 1650 7050 50  0001 C CNN

Commit message: rf layout
Parts:
- added C?: C, Capacitor_SMD:C_0603_1608Metric_Pad1.05x0.95mm_HandSolder, symbol Device:C
Connections:
- net +3V3: now also C?.1
- net GND: now also C?.2
Changed lines of the file:
@@
 	1    0    0    -1
 $EndComp
+$Comp
+L Device:C C?
+U 1 1 5F3FC447
+P 4900 1000
+F 0 "C?" H 5015 1046 50  0000 L CNN
+F 1 "C" H 5015 955 50  0000 L CNN
+F 2 "Capacitor_SMD:C_0603_1608Metric_Pad1.05x0.95mm_HandSolder" H 4938 850 50  0001 C CNN
+F 3 "~" H 4900 1000 50  0001 C CNN
+	1    4900 1000
+	1    0    0    -1
+$EndComp
+Wire Wire Line
+	4500 850  4900 850
+Connection ~ 4500 850
+Wire Wire Line
+	4900 1150 4900 1200
+Wire Wire Line
+	4900 1200 4500 1200
+Connection ~ 4500 1200
 $EndSCHEMATC

Commit message: rf layout:
Parts:
- 1.5pF1, 1pF1, 1pF2, 1pF3, 2.7nH1, 3.9nH1, 8.2nH1: footprint Capacitor_SMD:C_0402_1005Metric -> Capacitor_SMD:C_0603_1608Metric
- gave numbers to parts that had none: 1
Changed lines of the file:
@@
 F 0 "1.5pF1" V 10352 1800 50  0000 C CNN
 F 1 "C" V 10261 1800 50  0000 C CNN
-F 2 "Capacitor_SMD:C_0402_1005Metric" H 10138 1650 50  0001 C CNN
+F 2 "Capacitor_SMD:C_0603_1608Metric" H 10138 1650 50  0001 C CNN
 F 3 "~" H 10100 1800 50  0001 C CNN
 	1    10100 1800
@@
 F 0 "8.2nH1" H 9353 1996 50  0000 L CNN
 F 1 "L" H 9353 1905 50  0000 L CNN
-F 2 "Capacitor_SMD:C_0402_1005Metric" H 9300 1950 50  0001 C CNN
+F 2 "Capacitor_SMD:C_0603_1608Metric" H 9300 1950 50  0001 C CNN
 F 3 "~" H 9300 1950 50  0001 C CNN
 	1    9300 1950
@@
 F 0 "3.9nH1" V 9840 1800 50  0000 C CNN
 F 1 "L" V 9749 1800 50  0000 C CNN
-F 2 "Capacitor_SMD:C_0402_1005Metric" H 9650 1800 50  0001 C CNN
+F 2 "Capacitor_SMD:C_0603_1608Metric" H 9650 1800 50  0001 C CNN
 F 3 "~" H 9650 1800 50  0001 C CNN
 	1    9650 1800
@@
 F 0 "1pF2" H 10515 1996 50  0000 L CNN
 F 1 "C" H 10515 1905 50  0000 L CNN
-F 2 "Capacitor_SMD:C_0402_1005Metric" H 10438 1800 50  0001 C CNN
+F 2 "Capacitor_SMD:C_0603_1608Metric" H 10438 1800 50  0001 C CNN
 F 3 "~" H 10400 1950 50  0001 C CNN
 	1    10400 1950
@@
 F 0 "1pF3" H 10665 2696 50  0000 L CNN
 F 1 "C" H 10665 2605 50  0000 L CNN
-F 2 "Capacitor_SMD:C_0402_1005Metric" H 10588 2500 50  0001 C CNN
+F 2 "Capacitor_SMD:C_0603_1608Metric" H 10588 2500 50  0001 C CNN
 F 3 "~" H 10550 2650 50  0001 C CNN
 	1    10550 2650
@@
 F 0 "1pF1" H 10265 2696 50  0000 L CNN
 F 1 "C" H 10265 2605 50  0000 L CNN
-F 2 "Capacitor_SMD:C_0402_1005Metric" H 10188 2500 50  0001 C CNN
+F 2 "Capacitor_SMD:C_0603_1608Metric" H 10188 2500 50  0001 C CNN
 F 3 "~" H 10150 2650 50  0001 C CNN
 	1    10150 2650
@@
 F 0 "2.7nH1" V 9840 2100 50  0000 C CNN
 F 1 "L" V 9749 2100 50  0000 C CNN
-F 2 "Capacitor_SMD:C_0402_1005Metric" H 9650 2100 50  0001 C CNN
+F 2 "Capacitor_SMD:C_0603_1608Metric" H 9650 2100 50  0001 C CNN
 F 3 "~" H 9650 2100 50  0001 C CNN
 	1    9650 2100
@@
 $EndComp
 $Comp
-L Device:C C?
+L Device:C C15
 U 1 1 5F3FC447
 P 4900 1000
-F 0 "C?" H 5015 1046 50  0000 L CNN
+F 0 "C15" H 5015 1046 50  0000 L CNN
 F 1 "C" H 5015 955 50  0000 L CNN
 F 2 "Capacitor_SMD:C_0603_1608Metric_Pad1.05x0.95mm_HandSolder" H 4938 850 50  0001 C CNN

Commit message: add alot
Parts:
- added U?: NRF24L01_Breakout, RF_Module:nRF24L01_Breakout, symbol RF:NRF24L01_Breakout
Connections:
- net +3V3: now also U?.2 (VCC)
- net CE: now also U?.3 (CE)
- net CSN: now also U?.4 (~CSN)
- net GND: now also U?.1 (GND)
- net IRQ: now also U?.8 (IRQ)
- net MISO: now also U?.7 (MISO)
- net MOSI: now also U?.6 (MOSI)
- net SCK: now also U?.5 (SCK)
Changed lines of the file:
@@
 	4900 1200 4500 1200
 Connection ~ 4500 1200
+$Comp
+L RF:NRF24L01_Breakout U?
+U 1 1 5F40A6BF
+P 7350 5200
+F 0 "U?" H 7730 5246 50  0000 L CNN
+F 1 "NRF24L01_Breakout" H 7730 5155 50  0000 L CNN
+F 2 "RF_Module:nRF24L01_Breakout" H 7500 5800 50  0001 L CIN
+F 3 "http://www.nordicsemi.com/eng/content/download/2730/34105/file/nRF24L01_Product_Specification_v2_0.pdf" H 7350 5100 50  0001 C CNN
+	1    7350 5200
+	1    0    0    -1
+$EndComp
+Wire Wire Line
+	7350 4600 7350 4350
+$Comp
+L power:+3.3V #PWR?
+U 1 1 5F40BF56
+P 7350 4350
+F 0 "#PWR?" H 7350 4200 50  0001 C CNN
+F 1 "+3.3V" H 7365 4523 50  0000 C CNN
+F 2 "" H 7350 4350 50  0001 C CNN
+F 3 "" H 7350 4350 50  0001 C CNN
+	1    7350 4350
+	1    0    0    -1
+$EndComp
+Text GLabel 6700 5400 0    50   Input ~ 0
+CE
+Text GLabel 6700 5200 0    50   Input ~ 0
+CSN
+Text GLabel 6700 5100 0    50   Input ~ 0
+SCK
+Text GLabel 6700 5000 0    50   Input ~ 0
+MISO
+Text GLabel 6700 4900 0    50   Input ~ 0
+MOSI
+Wire Wire Line
+	6700 5400 6850 5400
+Wire Wire Line
+	6700 5200 6850 5200
+Wire Wire Line
+	6850 5100 6700 5100
+Wire Wire Line
+	6700 5000 6850 5000
+Wire Wire Line
+	6700 4900 6850 4900
+Text GLabel 6700 5500 0    50   Input ~ 0
+IRQ
+Wire Wire Line
+	6700 5500 6850 5500
+$Comp
+L power:GND #PWR?
+U 1 1 5F451534
+P 7350 5800
+F 0 "#PWR?" H 7350 5550 50  0001 C CNN
+F 1 "GND" H 7355 5627 50  0000 C CNN
+F 2 "" H 7350 5800 50  0001 C CNN
+F 3 "" H 7350 5800 50  0001 C CNN
+	1    7350 5800
+	1    0    0    -1
+$EndComp
 $EndSCHEMATC
