File: RX_nrf24/RX_nrf24.kicad_pcb (KiCad board)
At the start: 2 copper layers, 50 x 25 mm, 54 parts, among them J1 USB_B_Micro, J2 Conn_01x03_Male, J3 Conn_Coaxial, J4 Conn_01x10_Male, J5 Conn_01x04_Female, SW1 SW_Push, U1 USBLC6-2SC6, U2 AMS1117-3.3, U3 STM32F103C8Tx, U4 RFX2401C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

Commit message: a
Parts:
- removed C15, C17, C18, C19, C21, C23, C24: C, Capacitor_SMD:C_0603_1608Metric_Pad1.05x0.95mm_HandSolder
- removed L1, L2: L, Capacitor_SMD:C_0603_1608Metric_Pad1.05x0.95mm_HandSolder
- removed R1: 1M, Resistor_SMD:R_0603_1608Metric_Pad1.05x0.95mm_HandSolder
- removed R4, R5: R, Resistor_SMD:R_0603_1608Metric_Pad1.05x0.95mm_HandSolder
- removed U4: RFX2401C, RF:QFN50P300X300X60-17N
- added J6: Conn_01x06_Male, Connector_JST:JST_ZE_SM06B-ZESS-TB_1x06-1MP_P1.50mm_Horizontal, B.Cu at (155.8, 102.5)
- added J7: Conn_01x10_Male, Connector_PinHeader_2.54mm:PinHeader_1x10_P2.54mm_Vertical, F.Cu at (151.5, 90.5)
- added J8: Conn_01x10_Male, Connector_PinHeader_2.54mm:PinHeader_1x10_P2.54mm_Vertical, F.Cu at (151.5, 88.0)
- 1pF1, 1pF3: footprint Capacitor_SMD:C_0603_1608Metric -> Capacitor_SMD:C_0402_1005Metric
- 2.7nH1: footprint Capacitor_SMD:C_0603_1608Metric_Pad1.05x0.95mm_HandSolder -> Capacitor_SMD:C_0402_1005Metric
- C4, C9: footprint Capacitor_Tantalum_SMD:CP_EIA-3528-12_Kemet-T_Pad1.50x2.35mm_HandSolder -> Capacitor_SMD:C_1206_3216Metric
- J1: footprint Connector_USB:USB_Micro-B_GCT_USB3076-30-A -> Connector_USB:USB_Micro-B_Molex_47346-0001
- J3: footprint Connector_Coaxial:SMA_Amphenol_132289_EdgeMount -> Connector_Coaxial:SMA_Amphenol_132203-12_Horizontal
- SW1: footprint Button_Switch_THT:SW_PUSH_6mm_H5mm -> Button_Switch_SMD:SW_Push_1P1T_NO_6x6mm_H9.5mm
- U2: value AMS1117-3.3 -> MCP1700-3302E_SOT23; footprint Package_TO_SOT_SMD:SOT-223-3_TabPin2 -> Package_TO_SOT_SMD:SOT-23
- moved C3 108.6 mm to (187.0, 88.9), turned to 90 degrees
- moved C1 94.5 mm to (182.9, 96.5), turned to 90 degrees
- moved C2 94.0 mm to (178.1, 96.4), turned to 270 degrees
- moved J4 92.2 mm to (174.3, 93.2), turned to 270 degrees
- moved 1pF3 82.7 mm to (197.7, 102.5), turned to 270 degrees
- moved R6 80.9 mm to (195.3, 94.1), turned to 90 degrees
- moved R2 78.0 mm to (187.0, 92.0), turned to 270 degrees
- moved 1pF1 76.6 mm to (196.7, 102.5), turned to 270 degrees
- moved C6 73.0 mm to (185.5, 98.9), turned to 270 degrees
- moved C20 71.4 mm to (194.0, 106.0), turned to 90 degrees
- moved C14 70.7 mm to (190.1, 96.5), turned to 180 degrees
- moved C16 69.4 mm to (193.4, 96.5)
- moved C8 69.4 mm to (175.3, 97.5)
- moved C11 62.5 mm to (175.3, 96.0)
- moved C7 61.0 mm to (184.0, 107.5), turned to 270 degrees
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Connections:
- J3 pad 1: Net-(C23-Pad1) -> RF_out
- U3 pad 10: Net-(U3-Pad10) -> P1
- U3 pad 11: Net-(U3-Pad11) -> P2
- U3 pad 12: Net-(U3-Pad12) -> P3
- U3 pad 13: Net-(U3-Pad13) -> P4
- U3 pad 14: Net-(U3-Pad14) -> P5
- U3 pad 15: Net-(U3-Pad15) -> P6
- U3 pad 16: Net-(U3-Pad16) -> P7
- U3 pad 17: Net-(U3-Pad17) -> P8
- U3 pad 18: Net-(U3-Pad18) -> P9
- U3 pad 19: Net-(U3-Pad19) -> P10
- U3 pad 21: Net-(U3-Pad21) -> UART3_TX
- U3 pad 22: Net-(U3-Pad22) -> UART3_RX
- U3 pad 26: Net-(U3-Pad26) -> UART3_CTS
- U3 pad 27: Net-(U3-Pad27) -> UART3_RTS
Routing:
- net GND: track 0.00 -> 31.7 mm, vias 0 -> 1
- net +3V3: track 0.00 -> 27.4 mm
- net P10: track 0.00 -> 27.4 mm
- net P9: track 0.00 -> 24.6 mm
- net P8: track 0.00 -> 21.9 mm
- net P7: track 0.00 -> 19.5 mm
- net USB_D-: track 0.00 -> 17.5 mm
- net USB_D+: track 0.00 -> 16.8 mm
- net P6: track 0.00 -> 16.0 mm
- net P5: track 0.00 -> 12.2 mm
- net D+: track 0.00 -> 10.9 mm
- net D-: track 0.00 -> 10.1 mm
- net SCK: track 0.00 -> 9.79 mm, vias 0 -> 2
- net P4: track 0.00 -> 9.60 mm
- net +5V: track 0.00 -> 9.24 mm
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Other:
- board size 50 x 25 mm -> 58.5 x 26.2 mm
- net class Default: clearance 0.2 -> 0.15
- rule trace_clearance: 0.2 -> 0.15
- rule trace_min: 0.2 -> 0.15

Commit message: a
Parts:
- moved C6 8.29 mm to (186.5, 107.1), turned to 0 degrees
- moved 1pF2 4.80 mm to (195.6, 103.2)
- moved J3 4.80 mm to (200.3, 102.7)
- moved C20 4.69 mm to (191.9, 110.2)
- moved C22 4.69 mm to (187.2, 110.2)
- moved R7 4.69 mm to (189.7, 107.9)
- moved Y2 4.69 mm to (189.5, 110.1)
- moved C7 4.60 mm to (179.6, 108.7)
- moved R6 4.52 mm to (191.7, 96.9)
- moved 1.5pF1 4.52 mm to (194.4, 102.8)
- moved 1pF1 4.52 mm to (193.1, 105.3)
- moved 1pF3 4.52 mm to (194.1, 105.3)
- moved 2.7nH1 4.52 mm to (192.1, 104.3)
- moved 3.9nH1 4.52 mm to (192.6, 102.8)
- moved 8.2nH1 4.52 mm to (191.2, 103.3)
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Routing:
- net IRQ: track 0.00 -> 8.37 mm
- net Net-(R7-Pad2): track 0.00 -> 7.09 mm
- net Net-(R7-Pad1): track 0.00 -> 5.43 mm
- net Net-(C20-Pad1): track 0.00 -> 1.56 mm
- net Net-(C22-Pad1): track 0.00 -> 1.53 mm
- net Net-(C2-Pad1): track 1.47 -> 0.00 mm
- net RF_out: track 7.05 -> 5.85 mm
- net USB_D-: track 17.5 -> 16.7 mm
- net CSN: track 8.15 -> 7.61 mm

Commit message: update pcb
Parts:
- moved J3 5.62 mm to (204.4, 98.9)
Routing:
- net RF_out: track 5.85 -> 12.0 mm

Commit message: update pcb
Parts:
- C11, C8: moved to B.Cu
- moved D1 12.6 mm to (172.5, 114.9)
- moved R3 12.6 mm to (172.4, 113.4)
- moved J2 12.3 mm to (157.1, 114.7)
- moved J5 12.3 mm to (167.6, 114.7)
- moved C4 8.42 mm to (151.5, 100.8)
- moved U2 8.42 mm to (155.6, 101.1)
- moved C5 8.42 mm to (153.2, 101.0)
- moved C9 8.42 mm to (158.5, 101.0)
- moved J1 7.65 mm to (154.4, 108.1)
- moved C7 6.39 mm to (173.6, 111.0), turned to 180 degrees
- moved C11 6.23 mm to (169.8, 98.9)
- moved J3 6.21 mm to (198.3, 99.9)
- moved C8 5.51 mm to (169.8, 97.6)
- moved U3 5.16 mm to (170.0, 105.1)
- moved C10 5.07 mm to (163.8, 108.1)
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Connections:
- U1 pad 2: Net-(U1-Pad2) -> GND
- U1 pad 5: Net-(U1-Pad5) -> +5V
Routing:
- net P10: track 27.4 -> 4.57 mm
- net P9: track 24.6 -> 1.98 mm
- net NRST: track 0.00 -> 14.0 mm
- net P8: track 21.9 -> 8.93 mm
- net P7: track 19.5 -> 7.19 mm
- net P6: track 16.0 -> 5.77 mm
- net D+: track 10.9 -> 3.28 mm
- net D-: track 10.1 -> 2.56 mm
- net P5: track 12.2 -> 4.79 mm
- net RF_out: track 12.0 -> 5.68 mm
- net +5V: track 9.24 -> 3.56 mm
- net P2: track 6.73 -> 1.27 mm
- net P4: track 9.60 -> 4.35 mm
- net +3V3: track 27.4 -> 31.9 mm
- net P1: track 7.49 -> 3.27 mm
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Other:
- board size 58.5 x 26.2 mm -> 53.1 x 30 mm

Commit message: layout
Parts:
- C11, C8: moved to F.Cu
- moved C1 2.81 mm to (176.2, 98.2)
- moved C2 2.81 mm to (171.5, 98.3)
- moved Y1 2.81 mm to (173.7, 98.3)
- moved C8 2.27 mm to (168.7, 99.6)
- moved D1 1.35 mm to (173.9, 114.9)
- moved R3 1.35 mm to (173.8, 113.4)
- moved C11 1.26 mm to (168.7, 98.2)
- moved C10 1.08 mm to (163.9, 109.2)
- moved C7 1.08 mm to (173.8, 112.1)
- moved U3 1.08 mm to (170.1, 106.2)
Routing:
- net USB_D+: track 13.9 -> 1.93 mm
- net USB_D-: track 13.9 -> 3.82 mm
- net NRST: track 14.0 -> 21.5 mm
- net +3V3: track 31.9 -> 38.0 mm
- net GND: track 30.1 -> 35.2 mm
- net Net-(U3-Pad6): track 0.00 -> 4.84 mm
- net Net-(U3-Pad5): track 2.61 -> 7.14 mm
- net P3: track 4.32 -> 0.00 mm
- net P1: track 3.27 -> 1.66 mm
- net Net-(C2-Pad1): track 0.00 -> 1.47 mm
- net P2: track 1.27 -> 0.00 mm
- net IRQ: track 8.99 -> 9.71 mm
- net MISO: track 8.21 -> 8.81 mm
