File: RX_nrf24/RX_nrf24.kicad_pcb (KiCad board)
At the start: 2 copper layers, 58.5 x 26.2 mm, 44 parts, among them J1 USB_B_Micro, J2 Conn_01x03_Male, J3 Conn_Coaxial, J4 Conn_01x10_Male, J5 Conn_01x04_Female, J6 Conn_01x06_Male, J7 Conn_01x10_Male, J8 Conn_01x10_Male, SW1 SW_Push, U1 USBLC6-2SC6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

Commit message: a
Parts:
- added C13: C, Capacitor_SMD:C_0603_1608Metric, F.Cu at (158.2, 106.2)
- added R1: R, Resistor_SMD:R_0603_1608Metric, F.Cu at (158.5, 111.2)
- C1, C2: footprint Capacitor_SMD:C_0603_1608Metric_Pad1.05x0.95mm_HandSolder -> Capacitor_SMD:C_0402_1005Metric
- C20, C22: footprint Capacitor_SMD:C_0603_1608Metric -> Capacitor_SMD:C_0402_1005Metric
- R7: footprint Resistor_SMD:R_0603_1608Metric_Pad1.05x0.95mm_HandSolder -> Resistor_SMD:R_0402_1005Metric
- moved J2 12.7 mm to (156.8, 115.0)
- moved J5 12.7 mm to (167.2, 115.0)
- moved R3 9.70 mm to (152.8, 103.5), turned to 180 degrees
- moved C4 8.75 mm to (151.2, 100.0)
- moved C5 8.75 mm to (152.8, 100.2)
- moved C9 8.75 mm to (158.2, 100.2)
- moved U2 8.75 mm to (155.2, 100.2)
- moved D1 8.75 mm to (156.0, 103.5)
- moved J1 8.50 mm to (153.8, 109.0)
- moved C1 4.37 mm to (178.8, 95.2), turned to 180 degrees
- moved J3 4.07 mm to (203.3, 100.0)
- moved U1 2.85 mm to (158.2, 108.8)
- moved Y1 2.61 mm to (177.9, 97.2)
- moved C7 2.48 mm to (178.8, 111.0), turned to 180 degrees
- moved C2 1.62 mm to (177.0, 95.2), turned to 0 degrees
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Connections:
- U1 pad 2: Net-(U1-Pad2) -> GND
- U1 pad 5: Net-(U1-Pad5) -> +5V
Routing:
- net BOOT0: track 0.00 -> 36.9 mm
- net SWCLK: track 0.00 -> 23.8 mm
- net SWDIO: track 0.00 -> 20.5 mm
- net P9: track 24.6 -> 6.27 mm
- net P10: track 27.4 -> 10.3 mm
- net USB_D-: track 16.7 -> 0.04 mm
- net P8: track 21.9 -> 5.36 mm
- net USB_D+: track 16.9 -> 1.93 mm
- net +5V: track 9.24 -> 23.0 mm, vias 0 -> 1
- net P7: track 19.5 -> 6.12 mm
- net P6: track 16.0 -> 3.11 mm
- net +3V3: track 27.4 -> 40.2 mm, vias 0 -> 1
- net UART3_RTS: track 3.41 -> 12.8 mm
- net D+: track 10.9 -> 2.23 mm
- net IRQ: track 8.37 -> 0.13 mm
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Other:
- board size 58.5 x 26.2 mm -> 58.5 x 30 mm
- net class USB added: clearance 0.15, trace_width 0.35, via_dia 0.8, via_drill 0.4

Commit message: add alot
Parts:
- moved C10 8.81 mm to (163.2, 101.1)
- moved C7 6.82 mm to (177.2, 104.4), turned to 270 degrees
- moved U3 5.11 mm to (170.1, 103.5), turned to 225 degrees
- moved 1.5pF1 3.57 mm to (191.3, 104.5)
- moved 1pF1 3.57 mm to (189.9, 107.0)
- moved 1pF3 3.57 mm to (191.0, 107.0)
- moved 2.7nH1 3.57 mm to (189.0, 106.0)
- moved 3.9nH1 3.57 mm to (189.5, 104.5)
- moved 8.2nH1 3.57 mm to (188.0, 104.9)
- moved C13 3.57 mm to (184.9, 98.7)
- moved C14 3.57 mm to (183.4, 101.0)
- moved C16 3.57 mm to (186.7, 101.0)
- moved C20 3.57 mm to (188.6, 110.7)
- moved C22 3.57 mm to (184.1, 110.7)
- moved C6 3.57 mm to (183.1, 108.7)
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Routing:
- net BOOT0: track 36.9 -> 0.00 mm, vias 1 -> 0
- net SWCLK: track 23.8 -> 0.00 mm
- net SWDIO: track 20.5 -> 0.00 mm
- net GND: track 36.8 -> 55.3 mm, vias 7 -> 10
- net +3V3: track 40.2 -> 58.7 mm, vias 1 -> 0
- net IRQ: track 0.13 -> 14.2 mm
- net P9: track 6.27 -> 19.7 mm
- net RF_out: track 0.46 -> 12.9 mm
- net P10: track 10.3 -> 22.2 mm
- net SCK: track 4.87 -> 15.1 mm
- net P8: track 5.36 -> 13.9 mm
- net MISO: track 4.78 -> 12.1 mm
- net MOSI: track 4.92 -> 11.8 mm
- net P6: track 3.11 -> 9.30 mm
- net P7: track 6.12 -> 11.6 mm
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