File: RX_nrf24/RX_nrf24.kicad_pcb (KiCad board)
At the start: 2 copper layers, 58.5 x 30 mm, 46 parts, among them J1 USB_B_Micro, J2 Conn_01x03_Male, J3 Conn_Coaxial, J4 Conn_01x10_Male, J5 Conn_01x04_Female, J6 Conn_01x06_Male, J7 Conn_01x10_Male, J8 Conn_01x10_Male, SW1 SW_Push, U1 USBLC6-2SC6, U2 MCP1700-3302E_SOT23, U3 STM32F103C8Tx, U5 nRF24L01P, Y1 Crystal_GND24, Y2 Crystal_GND24

Commit message: a
a
Parts:
- moved C10 0.78 mm to (163.2, 101.9)
Routing:
- net UART3_RX: track 13.0 -> 9.07 mm
- net UART3_TX: track 13.4 -> 10.2 mm
- net GND: track 55.3 -> 52.3 mm
- net +3V3: track 58.7 -> 60.0 mm
Changed lines of the file:
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@@
   )
   (module Capacitor_SMD:C_0603_1608Metric_Pad1.05x0.95mm_HandSolder (layer F.Cu)
-    (at 163.23 101.14 90)
+    (at 163.21 101.92 90)
     (descr "Capacitor SMD 0603 (1608 Metric), square (rectangular) end terminal, IPC_7351 nominal with elongated pad for handsoldering. (Body size source: http://www.tortai-tech.com/upload/download/2011102023233369053.pdf), generated with kicad-footprint-generator")
     (tags "capacitor handsolder")
@@
   (segment (start 175.75 95.8) (end 175.8 95.75) (width 0.25) (layer F.Cu) (net 3))
   (segment (start 175.75 97.05) (end 175.75 95.8) (width 0.25) (layer F.Cu) (net 3))
-  (segment (start 163.71407 100.265) (end 163.23 100.265) (width 0.25) (layer F.Cu) (net 3))
-  (segment (start 165.515678 102.066608) (end 163.71407 100.265) (width 0.25) (layer F.Cu) (net 3))
   (segment (start 165.515678 102.172658) (end 165.515678 102.066608) (width 0.25) (layer F.Cu) (net 3))
   (segment (start 175.208321 105.395289) (end 177.564711 105.395289) (width 0.25) (layer F.Cu) (net 3))
@@
   (segment (start 172.88 97.47) (end 172.88 95.97) (width 0.25) (layer F.Cu) (net 11))
   (segment (start 165.162124 102.526212) (end 165.162124 102.512124) (width 0.25) (layer F.Cu) (net 11))
-  (segment (start 164.665 102.015) (end 163.23 102.015) (width 0.25) (layer F.Cu) (net 11))
   (segment (start 165.162124 102.512124) (end 164.665 102.015) (width 0.25) (layer F.Cu) (net 11))
-  (segment (start 161.415 102.015) (end 158.15 98.75) (width 0.25) (layer F.Cu) (net 11))
-  (segment (start 163.23 102.015) (end 161.415 102.015) (width 0.25) (layer F.Cu) (net 11))
   (segment (start 176.126212 104.523788) (end 177.15 103.5) (width 0.25) (layer F.Cu) (net 11))
   (segment (start 174.937876 104.523788) (end 176.126212 104.523788) (width 0.25) (layer F.Cu) (net 11))
@@
   (segment (start 172.92092 97.46092) (end 172.92092 98.886314) (width 0.25) (layer F.Cu) (net 11))
   (segment (start 172.91 97.45) (end 172.92092 97.46092) (width 0.25) (layer F.Cu) (net 11))
+  (segment (start 162.345 101.93) (end 163.21 102.795) (width 0.15) (layer F.Cu) (net 11))
+  (segment (start 161.33 101.93) (end 162.345 101.93) (width 0.15) (layer F.Cu) (net 11))
+  (segment (start 161.33 101.93) (end 158.15 98.75) (width 0.25) (layer F.Cu) (net 11))
+  (segment (start 161.415 102.015) (end 161.33 101.93) (width 0.25) (layer F.Cu) (net 11))
+  (segment (start 163.21 102.795) (end 165.535 102.795) (width 0.15) (layer F.Cu) (net 11))
   (segment (start 188.355 111.405) (end 188.6 111.16) (width 0.15) (layer F.Cu) (net 12))
   (segment (start 187.225 111.405) (end 188.355 111.405) (width 0.15) (layer F.Cu) (net 12))
@@
   (segment (start 179.940698 107.625) (end 179.807849 107.757849) (width 0.25) (layer F.Cu) (net 44))
   (segment (start 159.5 100.25) (end 158.325 100.25) (width 0.15) (layer B.Cu) (net 55))
-  (segment (start 166.222785 101.465551) (end 167.247234 102.49) (width 0.25) (layer F.Cu) (net 55))
-  (segment (start 167.247234 102.49) (end 167.72 102.49) (width 0.25) (layer F.Cu) (net 55))
-  (segment (start 167.72 102.49) (end 167.72 102.49) (width 0.25) (layer F.Cu) (net 55))
-  (via (at 167.72 102.49) (size 0.8) (drill 0.4) (layers F.Cu B.Cu) (net 55))
-  (segment (start 167.72 102.49) (end 163.02 102.49) (width 0.15) (layer B.Cu) (net 55))
-  (segment (start 160.78 100.25) (end 158.325 100.25) (width 0.15) (layer B.Cu) (net 55))
-  (segment (start 163.02 102.49) (end 160.78 100.25) (width 0.15) (layer B.Cu) (net 55))
-  (segment (start 160.5 101.75) (end 158.325 101.75) (width 0.15) (layer B.Cu) (net 56))
-  (segment (start 165.869231 101.819105) (end 166.76 102.709874) (width 0.25) (layer F.Cu) (net 56))
-  (segment (start 166.76 102.709874) (end 166.76 103.21) (width 0.25) (layer F.Cu) (net 56))
-  (segment (start 166.76 103.21) (end 166.76 103.21) (width 0.25) (layer F.Cu) (net 56))
-  (via (at 166.76 103.21) (size 0.8) (drill 0.4) (layers F.Cu B.Cu) (net 56))
-  (segment (start 163.315722 103.21) (end 166.76 103.21) (width 0.15) (layer B.Cu) (net 56))
-  (segment (start 161.855722 101.75) (end 163.315722 103.21) (width 0.15) (layer B.Cu) (net 56))
-  (segment (start 158.325 101.75) (end 161.855722 101.75) (width 0.15) (layer B.Cu) (net 56))
+  (segment (start 164.272224 99.51499) (end 161.11501 99.51499) (width 0.15) (layer F.Cu) (net 55))
+  (segment (start 166.222785 101.465551) (end 164.272224 99.51499) (width 0.15) (layer F.Cu) (net 55))
+  (segment (start 161.11501 99.51499) (end 160.945 99.685) (width 0.15) (layer F.Cu) (net 55))
+  (segment (start 160.945 99.685) (end 160.91 99.72) (width 0.15) (layer F.Cu) (net 55))
+  (via (at 160.945 99.685) (size 0.8) (drill 0.4) (layers F.Cu B.Cu) (net 55))
+  (segment (start 160.38 100.25) (end 160.945 99.685) (width 0.15) (layer B.Cu) (net 55))
+  (segment (start 158.325 100.25) (end 160.38 100.25) (width 0.15) (layer B.Cu) (net 55))
+  (segment (start 165.869231 101.819105) (end 163.990126 99.94) (width 0.15) (layer F.Cu) (net 56))
+  (segment (start 163.910117 100.020009) (end 161.829991 100.020009) (width 0.15) (layer F.Cu) (net 56))
+  (segment (start 163.990126 99.94) (end 163.910117 100.020009) (width 0.15) (layer F.Cu) (net 56))
+  (segment (start 161.829991 100.020009) (end 161.2 100.65) (width 0.15) (layer F.Cu) (net 56))
+  (segment (start 161.2 100.65) (end 161.2 100.65) (width 0.15) (layer F.Cu) (net 56))
+  (via (at 161.2 100.65) (size 0.8) (drill 0.4) (layers F.Cu B.Cu) (net 56))
+  (segment (start 160.1 101.75) (end 161.2 100.65) (width 0.15) (layer B.Cu) (net 56))
+  (segment (start 158.325 101.75) (end 160.1 101.75) (width 0.15) (layer B.Cu) (net 56))
   (segment (start 161.5 103.25) (end 158.325 103.25) (width 0.15) (layer B.Cu) (net 57))
   (segment (start 165.047731 105.345289) (end 163.605289 105.345289) (width 0.15) (layer F.Cu) (net 57))

Commit message: rf layout
Parts:
- added C15: C, Capacitor_SMD:C_0603_1608Metric_Pad1.05x0.95mm_HandSolder, F.Cu at (168.1, 110.6)
- moved J2 17.6 mm to (174.3, 115.0)
- moved J3 4.24 mm to (199.2, 101.0)
- moved C1 1.91 mm to (178.9, 97.2)
- moved C2 1.91 mm to (177.2, 97.2)
- moved Y1 1.91 mm to (178.1, 99.0)
- moved J5 1.70 mm to (165.6, 114.9)
- moved R6 0.54 mm to (188.1, 98.3)
- moved C13 0.32 mm to (184.8, 98.4)
- moved C14 0.32 mm to (183.3, 100.7)
- moved C16 0.32 mm to (186.6, 100.7)
- moved C11 0.10 mm to (173.9, 96.0)
- moved C8 0.10 mm to (173.9, 97.5)
Routing:
- net +3V3: track 60.0 -> 80.2 mm
- net USB_D-: track 0.00 -> 9.64 mm
- net USB_D+: track 1.93 -> 11.5 mm
- net GND: track 52.3 -> 60.9 mm, vias 10 -> 9
- net BOOT0: track 0.00 -> 5.05 mm
- net P6: track 9.30 -> 14.1 mm
- net UART3_RTS: track 13.5 -> 9.33 mm
- net Net-(U3-Pad6): track 5.07 -> 0.96 mm
- net Net-(U3-Pad5): track 7.92 -> 4.44 mm
- net RF_out: track 12.9 -> 9.56 mm
- net UART3_CTS: track 11.6 -> 8.42 mm
- net P1: track 9.48 -> 8.72 mm
- net P2: track 6.20 -> 6.81 mm
Other:
- board size 58.5 x 30 mm -> 54.4 x 30 mm

Commit message: rf layout:
Parts:
- 1.5pF1, 1pF1, 1pF2, 1pF3, 2.7nH1, 3.9nH1, 8.2nH1: footprint Capacitor_SMD:C_0402_1005Metric -> Capacitor_SMD:C_0603_1608Metric
- moved 1pF2 6.68 mm to (198.7, 102.1)
- moved 1.5pF1 6.15 mm to (196.6, 101.3)
- moved 1pF1 5.74 mm to (195.1, 104.5), turned to 0 degrees
- moved J3 5.31 mm to (204.5, 101.3)
- moved C12 5.26 mm to (192.7, 96.0), turned to 90 degrees
- moved 3.9nH1 5.16 mm to (193.6, 101.3)
- moved 2.7nH1 4.46 mm to (192.8, 103.8)
- moved 8.2nH1 4.42 mm to (191.4, 102.1)
- moved 1pF3 4.25 mm to (195.1, 106.0), turned to 0 degrees
- moved C14 3.88 mm to (185.7, 97.6)
- moved C20 3.88 mm to (191.0, 107.6)
- moved C22 3.88 mm to (186.5, 107.6)
- moved C6 3.88 mm to (185.5, 105.6)
- moved R7 3.88 mm to (188.8, 105.6)
- moved U5 3.88 mm to (187.2, 101.4)
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Routing:
- net +3V3: track 80.2 -> 136.1 mm
- net NRST: track 0.00 -> 21.5 mm
- net GND: track 60.9 -> 78.1 mm, vias 9 -> 12
- net CSN: track 12.2 -> 18.0 mm
- net Net-(R6-Pad1): track 0.00 -> 5.41 mm
- net BOOT0: track 5.05 -> 0.00 mm
- net IRQ: track 14.2 -> 19.0 mm
- net Net-(U3-Pad6): track 0.96 -> 5.45 mm
- net MOSI: track 11.8 -> 16.2 mm
- net MISO: track 12.1 -> 16.4 mm
- net SCK: track 15.1 -> 18.7 mm
- net CE: track 11.7 -> 15.1 mm
- net Net-(U3-Pad5): track 4.44 -> 7.38 mm
- net TXEN: track 6.69 -> 9.00 mm
- net Net-(2.7nH1-Pad1): track 2.48 -> 4.26 mm
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Other:
- board size 54.4 x 30 mm -> 58.9 x 30 mm

Commit message: add alot
Parts:
- added U4: NRF24L01_Breakout, RF_Module:nRF24L01_Breakout, F.Cu at (181.1, 112.4)
- moved J5 15.1 mm to (150.5, 115.0), turned to 90 degrees
- moved J2 6.97 mm to (167.3, 115.0)
- moved C9 6.80 mm to (151.6, 98.2)
- moved R3 4.22 mm to (156.9, 102.8), turned to 0 degrees
- moved C4 3.48 mm to (152.6, 103.1), turned to 180 degrees
- moved U2 1.70 mm to (154.5, 98.7), turned to 270 degrees
- moved C5 1.28 mm to (152.3, 101.3), turned to 180 degrees
- moved D1 1.23 mm to (156.9, 104.4)
- moved J6 1.22 mm to (154.5, 102.5)
- moved J3 1.21 mm to (203.3, 101.2)
- moved C20 1.00 mm to (190.8, 108.6)
- moved Y2 1.00 mm to (188.6, 108.6)
- moved J1 1.00 mm to (152.8, 109.0)
- moved C22 0.98 mm to (186.4, 108.6)
- moved R7 0.96 mm to (188.5, 106.5)
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Routing:
- net +3V3: track 136.1 -> 207.0 mm, vias 0 -> 1
- net GND: track 78.1 -> 132.9 mm, vias 12 -> 38
- net SWCLK: track 0.25 -> 24.7 mm
- net SWDIO: track 0.00 -> 16.0 mm
- net BOOT0: track 0.00 -> 15.4 mm
- net MOSI: track 16.2 -> 23.8 mm, vias 0 -> 1
- net CSN: track 18.0 -> 25.5 mm, vias 0 -> 1
- net NRST: track 21.5 -> 28.5 mm
- net CE: track 15.1 -> 22.0 mm, vias 0 -> 1
- net MISO: track 16.4 -> 22.6 mm, vias 0 -> 1
- net +5V: track 23.0 -> 17.4 mm
- net SCK: track 18.7 -> 24.3 mm, vias 2 -> 3
- net IRQ: track 19.0 -> 24.5 mm, vias 0 -> 1
- net RF_out: track 11.2 -> 6.22 mm
- net UART3_RX: track 9.10 -> 13.3 mm
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- added copper zone on B.Cu, net GND
Other:
- board size 58.9 x 30 mm -> 60 x 30 mm
- net class Default: clearance 0.15 -> 0.2; via_dia 0.8 -> 0.6; via_drill 0.4 -> 0.3
- rule trace_clearance: 0.15 -> 0.2

Commit message: addd
Routing:
- net GND: track 132.9 -> 144.2 mm
- net P10: track 20.4 -> 19.4 mm
Changed lines of the file:
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@@
     (thickness 1.6)
     (drawings 21)
-    (tracks 585)
+    (tracks 586)
     (zones 0)
     (modules 48)
@@
   )
   (setup
-    (last_trace_width 0.15)
+    (last_trace_width 1)
     (user_trace_width 0.15)
     (user_trace_width 0.35)
@@
   (gr_line (start 150 86.5) (end 200 86.5) (layer Edge.Cuts) (width 0.05))
   (gr_line (start 200 116.5) (end 150 116.5) (layer Edge.Cuts) (width 0.05))
-  (via (at 157.08 98.7) (size 0.6) (drill 0.3) (layers F.Cu B.Cu) (net 3))
+  (via (at 156.71 97.7) (size 0.6) (drill 0.3) (layers F.Cu B.Cu) (net 3))
   (via (at 188.74 104.53) (size 0.6) (drill 0.3) (layers F.Cu B.Cu) (net 3))
   (via (at 191.88 108.14) (size 0.8) (drill 0.4) (layers F.Cu B.Cu) (net 3))
@@
   (via (at 180.46 97.64) (size 0.8) (drill 0.4) (layers F.Cu B.Cu) (net 3))
   (segment (start 151.5 88) (end 175.5 88) (width 1) (layer F.Cu) (net 3))
-  (segment (start 175.75 88.25) (end 177.275 88.25) (width 1) (layer F.Cu) (net 3))
-  (segment (start 175.5 88) (end 175.75 88.25) (width 1) (layer F.Cu) (net 3))
   (segment (start 174.98 97.72) (end 174.98 96.22) (width 0.15) (layer F.Cu) (net 3))
   (segment (start 187.18 103.3425) (end 187.18 104.019278) (width 0.15) (layer F.Cu) (net 3))
@@
   (segment (start 186.875 87.975) (end 187.1 87.75) (width 0.25) (layer F.Cu) (net 3))
   (segment (start 185.325 87.975) (end 186.875 87.975) (width 0.25) (layer F.Cu) (net 3))
-  (segment (start 187.1 87.75) (end 189.055 89.705) (width 0.25) (layer F.Cu) (net 3))
   (segment (start 188.605 96.355) (end 189.855 97.605) (width 0.25) (layer F.Cu) (net 3))
   (segment (start 188.605 95.305) (end 188.605 96.355) (width 0.25) (layer F.Cu) (net 3))
@@
   (segment (start 189.055 89.705) (end 190.3 90.95) (width 0.25) (layer F.Cu) (net 3))
   (via (at 189.055 89.705) (size 0.6) (drill 0.3) (layers F.Cu B.Cu) (net 3))
+  (segment (start 186.85 88) (end 187.1 87.75) (width 1) (layer F.Cu) (net 3))
+  (segment (start 174.36 88) (end 186.85 88) (width 1) (layer F.Cu) (net 3))
+  (segment (start 189.055 89.23) (end 189.055 89.705) (width 1) (layer F.Cu) (net 3))
+  (segment (start 187.575 87.75) (end 189.055 89.23) (width 1) (layer F.Cu) (net 3))
+  (segment (start 187.1 87.75) (end 187.575 87.75) (width 1) (layer F.Cu) (net 3))
   (segment (start 189.1175 102.405) (end 190.1325 103.42) (width 0.25) (layer F.Cu) (net 4))
   (segment (start 191.2125 104.5) (end 194.3275 104.5) (width 0.25) (layer F.Cu) (net 4))
@@
   (segment (start 155.91001 96.39001) (end 155.91999 96.39001) (width 0.15) (layer F.Cu) (net 20))
   (segment (start 154.41 94.89) (end 155.91001 96.39001) (width 0.15) (layer F.Cu) (net 20))
-  (segment (start 154.90001 96.39001) (end 155.91999 96.39001) (width 0.15) (layer F.Cu) (net 20))
   (segment (start 155.91999 96.39001) (end 156.21999 96.39001) (width 0.15) (layer F.Cu) (net 20))
   (segment (start 154.05 93) (end 156.475 95.425) (width 0.15) (layer F.Cu) (net 21))

Commit message: a
Routing:
- net GND: track 144.2 -> 142.4 mm, vias 38 -> 208
- added copper zone on F.Cu, net GND

Commit message: bao cao
Parts:
- added G***: LOGO, drone_v3:pusheen, B.Cu at (170.3, 103.2)
- +3.3V CLK DIO GND: renamed from J5
- moved C6 0.43 mm to (185.0, 105.8)
- renumbered J7 to 3.3v, J2 to BOOT, J8 to G, SW1 to NRST, U3 to STM32, U4 to nRF, U5 to nRF24
Routing:
- net GND: track 142.4 -> 151.4 mm, vias 208 -> 300
- net NRST: track 28.5 -> 36.5 mm, vias 0 -> 2
- net +3V3: track 207.0 -> 210.0 mm, vias 1 -> 2
- net MISO: track 22.6 -> 21.4 mm
- net UART3_RX: track 13.3 -> 12.2 mm
- net Net-(3.9nH1-Pad1): track 3.46 -> 4.09 mm
- added copper zone on F.Cu, net Net-(2.7nH1-Pad1)
- added copper zone on F.Cu, net Net-(3.9nH1-Pad1)
Other:
- board size 60 x 30 mm -> 58.6 x 30.7 mm
- net class Default: clearance 0.2 -> 0.15
- rule trace_clearance: 0.2 -> 0.15
