File: RX_nrf24/_autosave-RX_nrf24.sch (KiCad schematic (older format))
At the start: 45 parts, among them J1 USB_B_Micro, J2 Conn_01x03_Male, J3 Conn_Coaxial, J4 Conn_01x10_Male, J5 Conn_01x04_Female, J6 Conn_01x06_Male, J7 Conn_01x10_Male, J8 Conn_01x10_Male, SW1 SW_Push, U1 USBLC6-2SC6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

Commit message: rf layout
Parts:
- added C15: C, Capacitor_SMD:C_0603_1608Metric_Pad1.05x0.95mm_HandSolder, symbol Device:C
Connections:
- net +3V3: now also C15.1
- net GND: now also C15.2
Changed lines of the file:
@@
 	1    0    0    -1
 $EndComp
+$Comp
+L Device:C C15
+U 1 1 5F3FC447
+P 4900 1000
+F 0 "C15" H 5015 1046 50  0000 L CNN
+F 1 "C" H 5015 955 50  0000 L CNN
+F 2 "Capacitor_SMD:C_0603_1608Metric_Pad1.05x0.95mm_HandSolder" H 4938 850 50  0001 C CNN
+F 3 "~" H 4900 1000 50  0001 C CNN
+	1    4900 1000
+	1    0    0    -1
+$EndComp
+Wire Wire Line
+	4500 850  4900 850
+Connection ~ 4500 850
+Wire Wire Line
+	4900 1150 4900 1200
+Wire Wire Line
+	4900 1200 4500 1200
+Connection ~ 4500 1200
 $EndSCHEMATC
